File: xhp70-driver.sch (KiCad schematic (older format))
At the start: 27 parts, among them J1 LEMO2, J2 AVR-ISP-6, Q1 Q_NMOS_GDS, U1 AL8871Q, U2 ATtiny85-20SU, U3 L7805

Commit message: Updated routing and added thicker traces
Parts:
- U3: symbol Regulator_Linear:L7805 -> Regulator_Linear:AP2127N-3.3
Changed lines of the file:
@@
 $EndComp
 $Comp
-L Regulator_Linear:L7805 U3
+L Regulator_Linear:AP2127N-3.3 U3
 U 1 1 6039EB96
 P 1800 5650
